File: speaker-board/microcontroller_MCU.kicad_sch (KiCad schematic)
At the start: 0 parts

Commit message: update
Parts:
- added C1: 100n, Capacitor_SMD:C_0603_1608Metric, symbol Device:C
- added D1: ESD5Z3.3, Diode_SMD:D_SOD-523, symbol Diode:ESD5Zxx
- added R1: 10k, symbol Device:R
- added SW1: SW_SPDT, symbol Switch:SW_SPDT
- added SW2: 95C06B2GWRT, Button_Switch_SMD:SW_Push_1P1T_NO_6x6mm_H9.5mm, symbol Switch:SW_Push
- added U1: STM32H723ZGTx, Package_QFP:LQFP-144_20x20mm_P0.5mm, symbol MCU_ST_STM32H7:STM32H723ZGTx
Connections:
- new net: R1.1, SW1.2 (B)
- new net: U1.107 (VSS), U1.120 (VSS), U1.130 (VSS), U1.16 (VSS), U1.38 (VSS), U1.51 (VSS), U1.61 (VSS), U1.83 (VSS), U1.94 (VSS)
- new net +3.3V: SW1.3 (C)
- new net BOOT0: R1.2, U1.138 (BOOT0)
- new net GND: C1.2, D1.2 (A), SW1.1 (A), SW2.1
- new net NRST: C1.1, D1.1 (K), SW2.2, U1.25 (NRST)
Other:
- note added: "BOOT0"
- note added: "MCU RESET"
Changed lines of the file:
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@@
 	(generator "eeschema")
 	(generator_version "8.0")
-	(paper "A4")
-)
+	(paper "A3")
