File: speaker-board/bluetooth.kicad_sch (KiCad schematic)
At the start: 0 parts

Commit message: updates
Parts:
- added U3: Microchip_BM83, RF_Module:Microchip_BM83, symbol RF_Bluetooth:Microchip_BM83
Connections:
- new net +3.3V: U3.23 (BAT_IN)
- new net GND: U3.16 (GND), U3.50 (GND), U3.56 (GND), U3.57 (GND)
- new net UART_RX: U3.29 (P8_6/UART_RXD)
- new net UART_TX: U3.30 (P8_5/UART_TXD)

Commit message: update
Parts:
- added D1, D2: LED, symbol Device:LED
Connections:
- net +3.3V: now also D1.2 (A), D2.2 (A)
- net at U3.32 (LED1): now also D1.1 (K)
- net at U3.34 (LED2): now also D2.1 (K)

Commit message: updated
Connections:
- net I2S_DR1_BM83: now reaches U3.1 (DR1)
- net I2S_RFS1_BM83: now reaches U3.2 (RFS1)
- net I2S_SCLK_BM83: now reaches U3.3 (SCLK1)
- net I2S_DT1_BM83: now reaches U3.4 (DT1)
- net I2S_MCLK1_BM83: now reaches U3.5 (MCLK1)
Changed lines of the file:
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@@
+		)
+	)
+	(hierarchical_label "I2S_SCLK_BM83"
+		(shape input)
+		(at 121.92 82.55 180)
+		(fields_autoplaced yes)
+		(effects
+			(font
+				(size 1.27 1.27)
+			)
+			(justify right)
+		)
+	)
+	(hierarchical_label "I2S_DR1_BM83"
+		(shape input)
+		(at 121.92 77.47 180)
+		(fields_autoplaced yes)
+		(effects
+			(font
+				(size 1.27 1.27)
+			)
+			(justify right)
 		)
 	)
@@
 		)
 	)
+	(hierarchical_label "I2S_MCLK1_BM83"
+		(shape input)
+		(at 121.92 87.63 180)
+		(fields_autoplaced yes)
+		(effects
+			(font
+				(size 1.27 1.27)
+			)
+			(justify right)
+		)
+	)
+	(hierarchical_label "I2S_DT1_BM83"
+		(shape input)
+		(at 121.92 85.09 180)
+		(fields_autoplaced yes)
+		(effects
+			(font
+				(size 1.27 1.27)
+			)
+			(justify right)
+		)
+	)
 	(hierarchical_label "UART_TX"
 		(shape input)
@@
 		)
 	)
+	(hierarchical_label "I2S_RFS1_BM83"
+		(shape input)
+		(at 121.92 80.01 180)
+		(fields_autoplaced yes)
+		(effects
+			(font
+				(size 1.27 1.27)
+			)
+			(justify right)
+		)
+	)
