File: speaker-board/speaker-board.kicad_sch (KiCad schematic)
At the start: 0 parts

Commit message: update
Other:
- sheet Bluetooth ports: added UART_RX, UART_TX; removed none
Changed lines of the file:
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@@
+			)
+		)
+		(pin "UART_TX" input
+			(at 31.75 121.92 180)
+			(effects
+				(font
+					(size 1.27 1.27)
+				)
+				(justify left)
+			)
+		)
+		(pin "UART_RX" input
+			(at 31.75 127 180)
+			(effects
+				(font
+					(size 1.27 1.27)
+				)
+				(justify left)
 			)
 		)

Commit message: updated
Other:
- sheet Bluetooth ports: added I2S_DR1_BM83, I2S_DT1_BM83, I2S_MCLK1_BM83, I2S_RFS1_BM83, I2S_SCLK_BM83; removed none
Changed lines of the file:
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@@
 		)
 		(pin "UART_TX" input
-			(at 31.75 121.92 180)
+			(at 31.75 143.51 180)
 			(effects
 				(font
@@
 		)
 		(pin "UART_RX" input
-			(at 31.75 127 180)
+			(at 31.75 147.32 180)
 			(effects
 				(font
+					(size 1.27 1.27)
+				)
+				(justify left)
+			)
+		)
+		(pin "I2S_DR1_BM83" input
+			(at 31.75 118.11 180)
+			(effects
+				(font
+					(size 1.27 1.27)
+				)
+				(justify left)
+			)
+		)
+		(pin "I2S_RFS1_BM83" input
+			(at 31.75 120.65 180)
+			(effects
+				(font
+					(size 1.27 1.27)
+				)
+				(justify left)
+			)
+		)
+		(pin "I2S_SCLK_BM83" input
+			(at 31.75 123.19 180)
+			(effects
+				(font
+					(size 1.27 1.27)
+				)
+				(justify left)
+			)
+		)
+		(pin "I2S_DT1_BM83" input
+			(at 31.75 125.73 180)
+			(effects
+				(font
+					(size 1.27 1.27)
+				)
+				(justify left)
+			)
+		)
+		(pin "I2S_MCLK1_BM83" input
+			(at 31.75 128.27 180)
+			(effects
+				(font

Commit message: update
Other:
- added sheet Crossovers (untitled.kicad_sch)
- sheet Amplifier ports: added high_pass_1, high_pass_2, low_pass_1; removed none
Changed lines of the file:
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@@
 	(paper "A4")
+	(sheet
+		(at 203.2 31.115)
+		(size 33.02 57.785)
+		(fields_autoplaced yes)
+		(stroke
+			(width 0.1524)
+			(type solid)
+		)
+		(fill
+			(color 0 0 0 0.0000)
+		)
+		(property "Sheetname" "Crossovers"
+			(at 203.2 30.4034 0)
+			(effects
+				(font
+					(size 1.27 1.27)
+				)
+				(justify left bottom)
+			)
+		)
+		(property "Sheetfile" "untitled.kicad_sch"
+			(at 203.2 89.4846 0)
+			(effects
+				(font
+					(size 1.27 1.27)
+				)
+				(justify left top)
+			)
+		)
+		(pin "low_pass_1" input
+			(at 203.2 43.18 180)
+			(effects
+				(font
+					(size 1.27 1.27)
+				)
+				(justify left)
+			)
+		)
+		(pin "high_pass_2" input
+			(at 203.2 53.34 180)
+			(effects
+				(font
+					(size 1.27 1.27)
+				)
+				(justify left)
+			)
+		)
+		(pin "high_pass_1" input
+			(at 203.2 48.26 180)
+			(effects
+				(font
+					(size 1.27 1.27)
+				)
+				(justify left)
+			)
+		)
+		(instances
+			(project "speaker-board"
+				(path "/4d2291af-ba5f-4125-9b43-741823f4a2c8"
+					(page "8")
+				)
+			)
+		)
+	)
 	(sheet
 		(at 31.75 104.14)
@@
 			)
 		)
+		(pin "high_pass_1" input
+			(at 85.09 120.65 180)
+			(effects
+				(font
+					(size 1.27 1.27)
+				)
+				(justify left)
+			)
+		)
+		(pin "high_pass_2" input
+			(at 85.09 124.46 180)
+			(effects
+				(font
+					(size 1.27 1.27)
+				)
+				(justify left)
+			)
+		)
+		(pin "low_pass_1" input
+			(at 85.09 116.84 180)
+			(effects
+				(font
+					(size 1.27 1.27)
+				)
+				(justify left)
+			)
+		)
