File: speaker-board/speaker-board.kicad_sch (KiCad schematic)
At the start: 0 parts

Commit message: add footprints
Other:
- sheet Amplifier ports: added AMP_~{FAULT}, AMP_~{RESET}, INPUT_HIGH_N, INPUT_HIGH_P, INPUT_LOW_N, INPUT_LOW_P, SPEAKER_OUT_HIGH_N, SPEAKER_OUT_HIGH_P, SPEAKER_OUT_LOW_N, SPEAKER_OUT_LOW_P; removed high_pass_1, high_pass_2, low_pass_1
Changed lines of the file:
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@@
 			)
 		)
-		(pin "high_pass_1" input
-			(at 85.09 120.65 180)
+		(pin "INPUT_HIGH_P" input
+			(at 85.09 115.57 180)
 			(effects
 				(font
@@
 			)
 		)
-		(pin "high_pass_2" input
-			(at 85.09 124.46 180)
+		(pin "INPUT_LOW_P" input
+			(at 85.09 147.32 180)
 			(effects
 				(font
@@
 			)
 		)
-		(pin "low_pass_1" input
-			(at 85.09 116.84 180)
+		(pin "INPUT_LOW_N" input
+			(at 85.09 149.86 180)
 			(effects
 				(font
@@
 			)
 		)
+		(pin "AMP_~{RESET}" input
+			(at 85.09 132.08 180)
+			(effects
+				(font
+					(size 1.27 1.27)
+				)
+				(justify left)
+			)
+		)
+		(pin "SPEAKER_OUT_HIGH_P" output
+			(at 121.92 110.49 0)
+			(effects
+				(font
+					(size 1.27 1.27)
+				)
+				(justify right)
+			)
+		)
+		(pin "SPEAKER_OUT_HIGH_N" output
+			(at 121.92 113.03 0)
+			(effects
+				(font
+					(size 1.27 1.27)
+				)
+				(justify right)
+			)
+		)
+		(pin "AMP_~{FAULT}" input
+			(at 85.09 134.62 180)
+			(effects
+				(font
+					(size 1.27 1.27)
+				)
+				(justify left)
+			)
+		)
+		(pin "SPEAKER_OUT_LOW_P" output
+			(at 121.92 151.13 0)
+			(effects
+				(font
+					(size 1.27 1.27)
+				)
+				(justify right)
+			)
+		)
+		(pin "INPUT_HIGH_N" input
+			(at 85.09 118.11 180)
+			(effects
+				(font
+					(size 1.27 1.27)
+				)
+				(justify left)
+			)
+		)
+		(pin "SPEAKER_OUT_LOW_N" output
+			(at 121.92 153.67 0)
+			(effects
+				(font
+					(size 1.27 1.27)
+				)
+				(justify right)
+			)
+		)
