File: speaker-board/power_conversion.kicad_sch (KiCad schematic)
At the start: 0 parts

Commit message: power conversion
Parts:
- added C46: 2.2u, Capacitor_SMD:C_0603_1608Metric_Pad1.08x0.95mm_HandSolder, symbol Device:C
- added C47, C49: 4.7u, Capacitor_SMD:C_1206_3216Metric_Pad1.33x1.80mm_HandSolder, symbol Device:C
- added C48: 100n, Capacitor_SMD:C_0603_1608Metric_Pad1.08x0.95mm_HandSolder, symbol Device:C
- added C50, C51: 22u, Capacitor_SMD:C_0603_1608Metric_Pad1.08x0.95mm_HandSolder, symbol Device:C
- added C52: 10u, symbol Device:C
- added C53: 100n, symbol Device:C
- added C54, C56: 22u, symbol Device:C
- added C55: 56p, symbol Device:C
- added D10, D7, D8, D9: Green, Diode_SMD:D_0603_1608Metric, symbol Device:LED
- added D11, D6: UDD32C05L01, Diode_SMD:D_SOD-323, symbol shuttle_parts:PESD5V0X1BCSFYL
- added D3 (x2): D_Schottky, Diode_SMD:D_PowerDI-123, symbol Device:D_Schottky
- added D4: SMF26A, 0_LHRE_Footprints:SOD-123FL, symbol Diode:ESD5Zxx
- added D5: SP3205-01ETG, 0_LHRE_Footprints:SP320501ETG, symbol shuttle_parts:SP3205-01ETG
- added F1, F2, F3, F4: 1A, Fuse:Fuse_0603_1608Metric_Pad1.05x0.95mm_HandSolder, symbol Device:Fuse
- added L6: 6.8uH, Inductor_SMD:L_Changjiang_FTC404020S, symbol Device:L
- added L7: 10u, symbol Device:L
- added R16, R24: 100k, Resistor_SMD:R_0603_1608Metric_Pad0.98x0.95mm_HandSolder, symbol Device:R_Small
- added R17: 13.7k, Resistor_SMD:R_0603_1608Metric_Pad0.98x0.95mm_HandSolder, symbol Device:R_Small
- added R18: 249k, symbol Device:R
- added R19: 18k, symbol Device:R
- added R20: 47k, Resistor_SMD:R_0603_1608Metric_Pad0.98x0.95mm_HandSolder, symbol Device:R
- added R21, R23: 5.1k, Resistor_SMD:R_0603_1608Metric_Pad0.98x0.95mm_HandSolder, symbol Device:R
- added R22: 10k, Resistor_SMD:R_0603_1608Metric_Pad0.98x0.95mm_HandSolder, symbol Device:R
- added TP1: +24V, TestPoint:TestPoint_THTPad_D2.0mm_Drill1.0mm, symbol Connector:TestPoint
- added TP2: +5V, TestPoint:TestPoint_THTPad_1.5x1.5mm_Drill0.7mm, symbol Connector:TestPoint
- added TP3: +3V3, TestPoint:TestPoint_THTPad_1.5x1.5mm_Drill0.7mm, symbol Connector:TestPoint
- added TP4: +12V, TestPoint:TestPoint_THTPad_1.5x1.5mm_Drill0.7mm, symbol Connector:TestPoint
- added U4: LMR51430XDDCR, Package_TO_SOT_SMD:SOT-23-6_Handsoldering, symbol Regulator_Switching:LMR51430
- added U5: RT9013-33GB, Package_TO_SOT_SMD:SOT-23-5, symbol 0_LHRE_Symbols:RT9013-33GB
- added U6: AP63200WU, Package_TO_SOT_SMD:TSOT-23-6, symbol Regulator_Switching:AP63200WU
Connections:
- new net: C50.1, C51.1, D3.2 (A), L6.2, R16.1
- new net: C48.2, L6.1, U4.2 (SW)
- new net: R16.2, R17.1, U4.4 (FB)
- new net: C48.1, U4.6 (CB)
- new net: D8.2 (A), R24.2
- new net: C55.2, R18.2, R19.1, U6.1 (FB)
- new net: C53.1, L7.1, U6.5 (SW)
- new net: D10.2 (A), R21.1
- new net: D9.2 (A), R23.1
- new net: D7.2 (A), R20.1
- new net: C53.2, U6.6 (BST)
- new net: R22.1, R23.2
- new net +12V: D11.2, F4.2, R20.2, TP4.1
- new net +12V_Unfused: C54.1, C55.1, C56.1, F4.1, L7.2, R18.1
- new net +24V: C46.1, C52.1, D3.1 (K), R24.1, TP1.1, U4.3 (VIN), U4.5 (EN), U6.2 (EN), U6.3 (IN)
- new net +24VFused: D3.2 (A), D4.1 (K), F1.2
- new net +3V3: D5.1, F3.2, R21.2, TP3.1
- new net +3V3_Unfused: C49.2, F3.1, U5.5 (VOUT)
- new net +5V: C47.2, D6.2, F2.2, R22.2, TP2.1, U5.1 (VIN), U5.3 (EN)
- new net +5V_Unfused: D3.1 (K), F2.1
- new net 24V_Unprotected: F1.1
- new net GND: C46.2, C47.1, C49.1, C50.2, C51.2, C52.2, C54.2, C56.2, D10.1 (K), D11.1, D4.2 (A), D5.2, D6.1, D7.1 (K), D8.1 (K), D9.1 (K), R17.2, R19.2, U4.1 (GND), U5.2 (GND), U6.4 (GND)
- no-connect marks 0 -> 1
Other:
- note added: "(3/5/12/24)-2.2 / .0002"
- note added: "+24V to +5V Buck Converter"
- note added: "24V to 12V Buck Converter"
- note added: "LDO Steps Voltage Down from 5V to 3.3V"
- note added: "R1"
- note added: "R2"
- note added: "Revised Mar 21"
- note added: "Schottky Datasheet: @ 25°C and 300mA avg current draw ~= 250mV forward voltage Buck needs to output 5.25V: -> Using R_{FBT} = (V_{OUT} - V_{REF})/V_{REF} * R_{FBB} -> R_{FBT} = (5.25V - 1V)=/1V * (11kOhm) = 46.75kOhm (~47kOhm)"
- company: (none) -> Dhairya Gupta & Charan Pradeep
